File: full-can-programmer.kicad_pcb (KiCad board)
At the start: 2 copper layers, 18.9 x 10.9 mm, 7 parts, among them J1 Conn_01x04, U1 ATtiny85-20SU

Commit message: Add files via upload
Parts:
- removed G***: LOGO, SamacSys_Parts:kicad-logo-smaller
- removed REF**: OSHW-Logo2_7.3x6mm_SilkScreen, Symbol:OSHW-Logo2_7.3x6mm_SilkScreen
- added J2: Conn_01x04, Connector_PinHeader_2.54mm:PinHeader_1x04_P2.54mm_Vertical, F.Cu at (151.5, 83.9)
- C1, U1: moved to B.Cu
- moved S1 5.68 mm to (157.0, 89.5), turned to 0 degrees
- moved S2 5.63 mm to (157.0, 85.9), turned to 180 degrees
- moved U1 4.83 mm to (158.9, 87.7), turned to 90 degrees
- moved C1 0.19 mm to (145.3, 85.2)
Connections:
- net /SCL_5V renamed /SCK
- net /SDA_5V renamed /MOSI
- U1 pad 1: (no net) -> /RESET
- U1 pad 6: (no net) -> /MISO
Routing:
- net /RESET: track 0.00 -> 17.3 mm, vias 0 -> 1
- net GND: track 0.00 -> 12.0 mm, vias 1 -> 2
- net /MISO: track 0.00 -> 9.12 mm
- net /MOSI: track 4.17 -> 13.0 mm
- net /SCK: track 8.32 -> 16.0 mm
- net /SW_A: track 7.97 -> 2.71 mm, vias 0 -> 1
- net /VIN: track 14.7 -> 17.4 mm
- net /SW_B: track 9.39 -> 6.75 mm, vias 0 -> 1
Other:
- board text added: "MISO"
- board text added: "MOSI"
- board text added: "RST"
- board text added: "SCK"
- board text added: "v0.1"

Commit message: Add files via upload
Other:
- board text added: "JLCJLCJLCJLC"
